File: hardware/schematics/PowerDeliveryBoard.sch (EAGLE design)
At the start: 9 parts, among them IC1 7812T, IC2 7812T, J1 XT60-M

Commit message: update
Parts:
- added C1, C2: (no value), capacitor-wima:C2,5-3
- added J3: T2M-105-01-X-D-TH, T2M-105-01-X-D-TH:T2M-105-01-X-D-TH
- added R1: 10k, rcl:R-US_0204/7
- added U$1: CURRENTSENSOR, dac:CURRENTSENSOR
- R3: value 10k -> (none); device rcl:R-US_0204/2V -> resistor-shunt:BVS
Connections:
- new net N$1: J1.+, R3.2
- new net N$2: C2.1, U$1.VCC
- new net N$3: C1.1, U$1.VIOUT
- net 0: now also J3.04, R1.2, U$1.GND; no longer R3.2
- net VCC: now also C1.2, C2.2, J3.01, J3.02, J3.03, J3.05, J3.06, J3.07, J3.08, R1.1; no longer J1.+
Other:
- note removed: "Although the package footprints were the same, the pinout for the regulators were different last year. If we are using the same 3v3 reg then we will have to account for that. Look at the datasheet of whatever regualtor we are getting to check the exact pinout"
- note removed: "This resistor footprint looks small. Make sure we will be able to actually fit the resistors on the board"
- moved on the sheet: C5, C6, C7, C8, J1, R2

Commit message: changes from review
Parts:
- removed C1, C2: (no value), capacitor-wima:C2,5-3
- removed R3: (no value), resistor-shunt:BVS
- removed U$1: CURRENTSENSOR, dac:CURRENTSENSOR
- added C3: .1 uF, capacitor-wima:C2,5-3
- added C4: (no value), capacitor-wima:C2,5-3
- added U1: GENERIC-SOIC8MSGEQ7N-FILTER, SparkFun-Retired:GENERIC-SOIC8MSGEQ7N-FILTER
Connections:
- removed net N$1: J1.+, R3.2
- removed net N$2: C2.1, U$1.VCC
- removed net N$3: C1.1, U$1.VIOUT
- new net +3V3: C8.1, IC2.VO, R2.1
- new net +5V: C6.1, C7.1, IC1.VO, IC2.VI
- new net GND: C3.2, C4.1, J1.-, U1.5, U1.6
- new net N$4: C3.1, U1.8
- new net VI_OUT: C4.2, J3.01, U1.7
- new net V_BATT: C5.1, IC1.VI, U1.3, U1.4
- new net V_BATT_IN: J1.+, U1.1, U1.2
- net 0: no longer J1.-, U$1.GND
- net VCC: no longer C1.2, C2.2, C5.1, C6.1, C7.1, C8.1, IC1.VI, IC1.VO, IC2.VI, IC2.VO, J3.01, R2.1, R3.1
Other:
- moved on the sheet: J1

Commit message: power
Connections:
- removed net N$4: C3.1, U1.8
- net +5V: now also C3.1, U1.8
Changed lines of the file:
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@@
 <part name="C4" library="capacitor-wima" library_urn="urn:adsk.eagle:library:116" deviceset="C" device="2,5-3" package3d_urn="urn:adsk.eagle:package:5436/1"/>
 <part name="U$2" library="microbuilder" deviceset="GND" device=""/>
+<part name="P+1" library="supply1" deviceset="+5V" device=""/>
 </parts>
 <sheets>
@@
 <instance part="U$2" gate="G$1" x="24.13" y="-6.35" smashed="yes">
 <attribute name="VALUE" x="22.606" y="-8.89" size="1.27" layer="96"/>
+</instance>
+<instance part="P+1" gate="1" x="16.51" y="27.94" smashed="yes">
+<attribute name="VALUE" x="19.05" y="27.94" size="1.778" layer="96"/>
 </instance>
 </instances>
@@
 <wire x1="113.03" y1="25.4" x2="113.03" y2="27.94" width="0.1524" layer="91"/>
 </segment>
+<segment>
+<pinref part="U1" gate="G$1" pin="8"/>
+<pinref part="C3" gate="G$1" pin="1"/>
+<wire x1="17.78" y1="12.7" x2="17.78" y2="17.78" width="0.1524" layer="91"/>
+<wire x1="17.78" y1="17.78" x2="25.4" y2="17.78" width="0.1524" layer="91"/>
+<pinref part="P+1" gate="1" pin="+5V"/>
+<wire x1="16.51" y1="25.4" x2="16.51" y2="17.78" width="0.1524" layer="91"/>
+<wire x1="16.51" y1="17.78" x2="17.78" y2="17.78" width="0.1524" layer="91"/>
+<junction x="17.78" y="17.78"/>
+</segment>
 </net>
 <net name="+3V3" class="0">
@@
 </segment>
 </net>
-<net name="N$4" class="0">
-<segment>
-<pinref part="U1" gate="G$1" pin="8"/>
-<pinref part="C3" gate="G$1" pin="1"/>
-<wire x1="17.78" y1="12.7" x2="17.78" y2="17.78" width="0.1524" layer="91"/>
-<wire x1="17.78" y1="17.78" x2="25.4" y2="17.78" width="0.1524" layer="91"/>
-</segment>
-</net>
