File: hardware/schematics/GroundStation/Ground_Station_Board.brd (EAGLE design)
At the start: 100 x 66 mm, 11 parts

Commit message: board's smaller now
Parts:
- moved LED3 104.3 mm to (6.35, 20.3)
- moved LED2 95.7 mm to (6.35, 29.2)
- moved LED1 90.4 mm to (6.35, 38.1)
- moved R3 82.1 mm to (17.8, 19.1), turned to 0 degrees
- moved R2 72.8 mm to (17.8, 27.9), turned to 0 degrees
- moved R1 66.3 mm to (17.8, 36.8), turned to 0 degrees
- moved C1 56.2 mm to (8.89, 50.8), turned to 270 degrees
- moved C2 49.6 mm to (14.0, 50.8), turned to 270 degrees
- moved C3 42.4 mm to (20.3, 50.8), turned to 270 degrees
- moved U$2 6.35 mm to (40.6, 49.5)
- moved XBEE 6.35 mm to (14.0, 66.0), turned to 90 degrees
Connections:
- net +3V3: now also U$2.3V3; no longer U$2.3V3_LO
- net LED_1: now also U$2.24; no longer U$2.37/A18
- net LED_2: now also U$2.25; no longer U$2.38/A19
- net LED_3: now also U$2.26; no longer U$2.39/A20
- net XBEE_EN: now also U$2.3/CANTX; no longer U$2.22/A8
- net XBEE_RST: now also U$2.4/CANRX; no longer U$2.20/A6
Routing:
- net +3V3: track 69.6 -> 31.5 mm
- net LED_3: track 46.3 -> 20.0 mm
- net LED_2: track 41.2 -> 15.1 mm
- net XBEE_RST: track 46.6 -> 20.6 mm
- net XBEE_EN: track 47.7 -> 23.6 mm
- net LED_1: track 36.1 -> 12.5 mm
- net XBEE_RX: track 33.2 -> 27.7 mm
- net N$1: track 11.2 -> 7.62 mm
- net N$3: track 11.2 -> 7.62 mm
- net N$2: track 10.2 -> 7.62 mm
- net XBEE_TX: track 32.3 -> 30.8 mm
Other:
- board size 100 x 66 mm -> 50.5 x 66 mm
